Commit message: update

File: src/demo_world/urdf/blue_cube.urdf (robot description, URDF)
Before this commit: robot blue_cube, 1 links, 0 joints
Links:
- link base_link: mass 0.1 -> 0.0025; geometry collision box size=0.02 0.02 0.02; visual box size=0.02 0.02 0.02

File: src/demo_world/urdf/conveyor.urdf (robot description, URDF)
Before this commit: robot liukuhihna_gazebo, 3 links, 2 joints
Links:
- added link camera_link, mass 1e-5; collision box size=0.05 0.05 0.05; visual box size=0.05 0.05 0.05
- link belt_moving: geometry collision box size=0.425 2.4 0.001
- link belt_visual: geometry collision mesh filename=package://demo_world/meshes/conveyor_simple.stl scale=1 2 1; visual mesh filename=package://demo_world/meshes/conveyor_belt.stl scale=1 2 1
Joints:
- added joint camera_joint: type fixed, parent belt_visual, child camera_link, origin xyz=0.05 0 2.5 rpy=0 1.57 0, axis 0 1 0
- joint belt_joint: limit lower=0.0 upper=1 effort=1000 velocity=1000 -> lower=-1 upper=1 effort=1000 velocity=1000
